File: intg circt.kicad_sch (KiCad schematic)
At the start: 33 parts, among them J2 USB_C_Receptacle_USB2.0_16P, U1 ESP32-S3-MINI-1U, U2 MAXM86161EFD_T, U3 BMI270, U4 BQ24074RGT, U6 USBLC6-2P6, U7 MAX17048X+T10, U8 TLV75533PDBV

Commit message: temp sensor added, sd card schematic done, recheck.
Parts:
- added C14: 10pF, Capacitor_SMD:C_0201_0603Metric, symbol Device:C
- added C15: 100nF, Capacitor_SMD:C_0201_0603Metric, symbol Device:C
- added J1: Micro_SD_Card_Det_Hirose_DM3AT, Connector_Card:microSD_HC_Hirose_DM3AT-SF-PEJM5, symbol Connector:Micro_SD_Card_Det_Hirose_DM3AT
- added R12, R13, R14, R15, R16: 10kR, Resistor_SMD:R_0201_0603Metric, symbol Device:R
- added U5: TMP117xxDRV, Package_SON:WSON-6-1EP_2x2mm_P0.65mm_EP1x1.6mm, symbol Sensor_Temperature:TMP117xxDRV
Connections:
- net +3V3: now also C14.1, C15.1, J1.4 (VDD), R12.1, R13.1, R14.1, R15.1, R16.1
- net GND: now also C14.2, C15.2, J1.6 (VSS), J1.9 (DET_B), J1.SH (SHIELD)
- net IO15 renamed J1_CD
- net J1_CD: now also J1.2 (DAT3/CD), R12.2
- net IO16 renamed J1_CMD
- net J1_CMD: now also J1.3 (CMD), R13.2, R16.2
- net IO17 renamed J1_DAT0
- net J1_DAT0: now also J1.7 (DAT0), R14.2
- net IO18 renamed J1_DET_A
- net J1_DET_A: now also J1.10 (DET_A)
- net IO21: no longer names the net of U1.25 (IO21)
- new net J1_CLK: J1.5 (CLK)
- new net J1_DAT1: J1.8 (DAT1), R15.2
- new net J1_DAT2: J1.1 (DAT2)
Other:
- moved on the sheet: C5, C6, C7, C8, D2, R1, R2, R3, R4, R5, TH1, U4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

Commit message: I HAVE ADDED THE EDA SENSOR
Parts:
- removed U5: TMP117xxDRV, Package_SON:WSON-6-1EP_2x2mm_P0.65mm_EP1x1.6mm, symbol Sensor_Temperature:TMP117xxDRV
- added C16, C17, C18, C3: 0.1uF, Capacitor_SMD:C_0201_0603Metric, symbol Device:C
- added J3: Conn_01x02_Pin, Connector_PinHeader_1.00mm:PinHeader_1x02_P1.00mm_Vertical, symbol Connector:Conn_01x02_Pin
- added R17, R19, R20, R21: 100KR, Resistor_SMD:R_0201_0603Metric, symbol Device:R
- added R18: 1MR, Resistor_SMD:R_0201_0603Metric, symbol Device:R
- added U9: LMV358IDR, footprints:LMV358IDR, symbol LMV358IDR:LMV358IDR
Connections:
- net +3V3: now also C18.1, J3.1 (Pin_1), R21.1, U9.8 (V+)
- net GND: now also C17.2, C18.2, R20.2, U9.4 (V-)
- new net: C17.1, R20.1, R21.2, U9.5 (INB+)
- new net INB-: C16.2, R17.2, R19.2, U9.6 (INB-)
- new net OUT_A: C3.2, R17.1, R18.2, U9.1 (OUT_A)
- new net OUT_B: C16.1, R19.1, U9.3 (INA+), U9.7 (OUT_B)
- new net skin++: C3.1, J3.2 (Pin_2), R18.1, U9.2 (INA-)
Other:
- moved on the sheet: D2, R4, R5, U8

Commit message: new library
Parts:
- removed J1: Micro_SD_Card_Det_Hirose_DM3AT, Connector_Card:microSD_HC_Hirose_DM3AT-SF-PEJM5, symbol Connector:Micro_SD_Card_Det_Hirose_DM3AT
- added J4: 5033981892, CONN_503398-1892_MOL, symbol KiCADv6:5033981892
Connections:
- net +3V3: now also J4.4 (VDD)
- net GND: now also J4.6 (VSS)
- net J1_CD: now also J4.2 (CD/DAT3)
- net J1_CLK: now also J4.5 (CLK)
- net J1_CMD: now also J4.3 (CMD)
- net J1_DAT0: now also J4.7 (DA0)
- net J1_DAT1: now also J4.8 (DAT1)
- net J1_DAT2: now also J4.1 (DAT2)
- no-connect marks 10 -> 12
Changed lines of the file:
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@@
 	)
 	(no_connect
+		(at 46.99 269.24)
+	)
+	(no_connect
+		(at 46.99 266.7)
+	)
+	(no_connect
 		(at 66.04 157.48)
 	)
@@
 		)
 	)
-	(label "J1_DET_A"
-		(at 46.99 266.7 180)
-		(effects
-			(font
-				(size 1.27 1.27)
-			)
-			(justify right bottom)
-		)
-	)
 	(label "OUT_B"
 		(at 177.8 228.6 0)
@@
 	)
 	(symbol
-		(lib_id "power:GND")
-		(at 90.17 269.24 90)
-		(mirror x)
-		(unit 1)
-		(body_style 1)
-		(exclude_from_sim no)
-		(in_bom yes)
-		(on_board yes)
-		(in_pos_files yes)
-		(dnp no)
-		(fields_autoplaced yes)
-		(property "Reference" "#PWR052"
-			(at 96.52 269.24 0)
-			(hide yes)
-			(show_name no)
-			(do_not_autoplace no)
-			(effects
-				(font
-					(size 1.27 1.27)
-				)
-			)
-		)
-		(property "Value" "GND"
-			(at 93.98 269.2399 90)
-			(show_name no)
-			(do_not_autoplace no)
-			(effects
-				(font
-					(size 1.27 1.27)
-				)
-				(justify right)
-			)
-		)
-		(property "Footprint" ""
-			(at 90.17 269.24 0)
-			(hide yes)
-			(show_name no)
-			(do_not_autoplace no)
-			(effects
-				(font
-					(size 1.27 1.27)
-				)
-			)
-		)
-		(property "Datasheet" ""
-			(at 90.17 269.24 0)
-			(hide yes)
-			(show_name no)
-			(do_not_autoplace no)
-			(effects
-				(font
-					(size 1.27 1.27)
-				)
-			)
-		)
-		(property "Description" "Power symbol creates a global label with name \"GND\" , ground"
-			(at 90.17 269.24 0)
-			(hide yes)
-			(show_name no)
-			(do_not_autoplace no)
-			(effects
-				(font
-					(size 1.27 1.27)
-				)
-			)
-		)
-		(pin "1"
-		)
-		(instances
-			(project "intg circt"
-				(path "/f86b7e7a-57ea-4a2f-9196-86e87a059a37"
-					(reference "#PWR052")
-					(unit 1)
-				)
-			)
-		)
-	)
-	(symbol
-		(lib_id "power:GND")
-		(at 46.99 269.24 270)
-		(mirror x)
-		(unit 1)
-		(body_style 1)
-		(exclude_from_sim no)
-		(in_bom yes)
-		(on_board yes)
-		(in_pos_files yes)
-		(dnp no)
-		(fields_autoplaced yes)
-		(property "Reference" "#PWR054"
-			(at 40.64 269.24 0)
-			(hide yes)
-			(show_name no)
-			(do_not_autoplace no)
-			(effects
-				(font
-					(size 1.27 1.27)
-				)
-			)
-		)
-		(property "Value" "GND"
-			(at 43.18 269.2399 90)
-			(show_name no)
-			(do_not_autoplace no)
-			(effects
-				(font
-					(size 1.27 1.27)
-				)
-				(justify right)
-			)
-		)
-		(property "Footprint" ""
-			(at 46.99 269.24 0)
-			(hide yes)
-			(show_name no)
-			(do_not_autoplace no)
-			(effects
-				(font
-					(size 1.27 1.27)
-				)
-			)
-		)
-		(property "Datasheet" ""
-			(at 46.99 269.24 0)
-			(hide yes)
-			(show_name no)
-			(do_not_autoplace no)
-			(effects
-				(font
-					(size 1.27 1.27)
-				)
-			)
-		)
-		(property "Description" "Power symbol creates a global label with name \"GND\" , ground"
-			(at 46.99 269.24 0)
-			(hide yes)
-			(show_name no)
-			(do_not_autoplace no)
-			(effects
-				(font
-					(size 1.27 1.27)
-				)
-			)
-		)
-		(pin "1"
-		)
-		(instances
-			(project "intg circt"
-				(path "/f86b7e7a-57ea-4a2f-9196-86e87a059a37"
-					(reference "#PWR054")
-					(unit 1)
-				)
-			)
-		)
-	)
-	(symbol
 		(lib_id "Device:C")
 		(at 166.37 213.36 90)
@@
 	)
 	(symbol
-		(lib_id "Connector:Micro_SD_Card_Det_Hirose_DM3AT")
-		(at 69.85 256.54 0)
-		(unit 1)
-		(body_style 1)
-		(exclude_from_sim no)
-		(in_bom yes)
-		(on_board yes)
-		(in_pos_files yes)
-		(dnp no)
-		(fields_autoplaced yes)
-		(property "Reference" "J1"
-			(at 70.485 234.95 0)
-			(show_name no)
-			(do_not_autoplace no)
-			(effects
-				(font
-					(size 1.27 1.27)
-				)
-			)
-		)
-		(property "Value" "Micro_SD_Card_Det_Hirose_DM3AT"
-			(at 70.485 237.49 0)
-			(show_name no)
-			(do_not_autoplace no)
-			(effects
-				(font
-					(size 1.27 1.27)
-				)
-			)
-		)
-		(property "Footprint" "Connector_Card:microSD_HC_Hirose_DM3AT-SF-PEJM5"
-			(at 121.92 238.76 0)
-			(hide yes)
-			(show_name no)
-			(do_not_autoplace no)
-			(effects
-				(font
-					(size 1.27 1.27)
-				)
-			)
-		)
-		(property "Datasheet" "https://www.hirose.com/product/en/download_file/key_name/DM3/category/Catalog/doc_file_id/49662/?file_category_id=4&item_id=195&is_series=1"
-			(at 69.85 254 0)
-			(hide yes)
-			(show_name no)
-			(do_not_autoplace no)
-			(effects
-				(font
-					(size 1.27 1.27)
-				)
-			)
-		)
-		(property "Description" "Micro SD Card Socket with card detection pins"
-			(at 69.85 256.54 0)
-			(hide yes)
-			(show_name no)
-			(do_not_autoplace no)
-			(effects
-				(font
-					(size 1.27 1.27)
-				)
-			)
-		)
-		(property "MPN" "https://www.lioncircuits.com/parts/DM3AT-SF-PEJM5"
-			(at 69.85 256.54 0)
-			(hide yes)
-			(show_name no)
-			(do_not_autoplace no)
-			(effects
-				(font
-					(size 1.27 1.27)
-				)
-			)
-		)
-		(pin "SH"
-		)
-		(pin "1"
-		)
-		(pin "9"
-		)
-		(pin "5"
-		)
-		(pin "3"
-		)
-		(pin "10"
-		)
-		(pin "8"
-		)
-		(pin "2"
-		)
-		(pin "4"
-		)
-		(pin "6"
-		)
-		(pin "7"
-		)
-		(instances
-			(project "intg circt"
-				(path "/f86b7e7a-57ea-4a2f-9196-86e87a059a37"
-					(reference "J1")
-					(unit 1)
-				)
-			)
-		)
-	)
-	(symbol
 		(lib_id "Device:R")
 		(at 170.18 222.25 90)
@@
 					(unit 1)
 				)
+			)
+		)
+	)
+	(symbol
+		(lib_id "KiCADv6:5033981892")
+		(at 46.99 246.38 0)
+		(unit 1)
+		(body_style 1)
+		(exclude_from_sim no)
+		(in_bom yes)
+		(on_board yes)
+		(in_pos_files yes)
+		(dnp no)
+		(fields_autoplaced yes)
+		(property "Reference" "J4"
+			(at 60.96 256.5399 0)
+			(show_name no)
+			(do_not_autoplace no)
+			(effects
+				(font
+					(size 1.524 1.524)
+				)
+				(justify left)
+			)
+		)
+		(property "Value" "5033981892"
+			(at 60.96 259.0799 0)
+			(show_name no)
+			(do_not_autoplace no)
+			(effects
+				(font
+					(size 1.524 1.524)
+				)
+				(justify left)
+			)
+		)
+		(property "Footprint" "CONN_503398-1892_MOL"
+			(at 46.99 246.38 0)
+			(hide yes)
+			(show_name no)
+			(do_not_autoplace no)
+			(effects
+				(font
+					(size 1.27 1.27)
+					(italic yes)
+				)
+			)
+		)
+		(property "Datasheet" "https://www.molex.com/en-us/products/part-detail-pdf/5033981892?display=pdf"
+			(at 46.99 246.38 0)
+			(hide yes)
+			(show_name no)
+			(do_not_autoplace no)
+			(effects
+				(font
+					(size 1.27 1.27)
+					(italic yes)
+				)
+			)
+		)
+		(property "Description" ""
+			(at 46.99 246.38 0)
+			(hide yes)
+			(show_name no)
+			(do_not_autoplace no)
+			(effects
+				(font
+					(size 1.27 1.27)
+				)
+			)
+		)
+		(pin "6"
+		)
+		(pin "3"
+		)
+		(pin "4"
+		)
+		(pin "9"
+		)
+		(pin "10"
+		)
+		(pin "1"
+		)
+		(pin "8"
+		)
+		(pin "7"
+		)
+		(pin "2"
+		)
+		(pin "5"
+		)
+		(instances
+			(project "intg circt"
+				(path "/f86b7e7a-57ea-4a2f-9196-86e87a059a37"
+					(reference "J4")
+					(unit 1)
+				)

Commit message: change so much
Parts:
- added J1, J6: Conn_01x01_Pin, Connector_PinHeader_1.00mm:PinHeader_1x01_P1.00mm_Vertical, symbol Connector:Conn_01x01_Pin
- added J5: Conn_01x02_Pin, Connector_PinHeader_1.00mm:PinHeader_1x02_P1.00mm_Vertical, symbol Connector:Conn_01x02_Pin
Connections:
- net IO6 is gone; now on net OUT_A: U1.10 (IO6)
- net IO7 is gone; now on net OUT_B: U1.11 (IO7)
- net +3V3: now also J6.1 (Pin_1)
- net GND: now also J1.1 (Pin_1)
- net Temp_SDA: now reaches U1.25 (IO21)
- net Temp_SDA: now also J5.1 (Pin_1)
- net IO26 renamed Temp_SCL
- net Temp_SCL: now also J5.2 (Pin_2)
Other:
- moved on the sheet: C16, C17, C18, C3, J3, R17, R18, R19, R20, R21, U9
