File: intg circt.kicad_pcb (KiCad board)
At the start: 2 copper layers, 16.8 x 23.9 mm, 33 parts, among them J2 USB_C_Receptacle_USB2.0_16P, U1 ESP32-S3-MINI-1U, U2 MAXM86161EFD_T, U3 BMI270, U4 BQ24074RGT, U6 USBLC6-2P6, U7 MAX17048X+T10, U8 TLV75533PDBV

Commit message: change
Parts:
- moved J2 0.10 mm to (76.8, 62.7)
Changed lines of the file:
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@@
 	(footprint "Connector_USB:USB_C_Receptacle_GCT_USB4105-xx-A_16P_TopMnt_Horizontal"
 		(layer "F.Cu")
-		(at 76.8 62.59)
+		(at 76.75 62.68)
 		(descr "USB 2.0 Type C Receptacle, GCT, 16P, top mounted, horizontal, 5A: https://gct.co/files/drawings/usb4105.pdf")
 		(tags "USB C Type-C Receptacle SMD USB 2.0 16P 16C USB4105-15-A USB4105-15-A-060 USB4105-15-A-120 USB4105-GF-A USB4105-GF-A-060 USB4105-GF-A-120")

Commit message: just tested if it works, it does i think
Parts:
- moved J2 0.18 mm to (76.8, 62.5)
Changed lines of the file:
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@@
 	(footprint "Connector_USB:USB_C_Receptacle_GCT_USB4105-xx-A_16P_TopMnt_Horizontal"
 		(layer "F.Cu")
-		(at 76.75 62.68)
+		(at 76.75 62.5)
 		(descr "USB 2.0 Type C Receptacle, GCT, 16P, top mounted, horizontal, 5A: https://gct.co/files/drawings/usb4105.pdf")
 		(tags "USB C Type-C Receptacle SMD USB 2.0 16P 16C USB4105-15-A USB4105-15-A-060 USB4105-15-A-120 USB4105-GF-A USB4105-GF-A-060 USB4105-GF-A-120")

Commit message: I HAVE ADDED THE EDA SENSOR
Parts:
- added C14: 10pF, Capacitor_SMD:C_0201_0603Metric, F.Cu at (114.5, 47.2)
- added C15: 100nF, Capacitor_SMD:C_0201_0603Metric, F.Cu at (114.5, 49.0)
- added C16, C3: 0.1uF, Capacitor_SMD:C_0201_0603Metric, F.Cu at (97.8, 47.2)
- added C17: 0.1uF, Capacitor_SMD:C_0201_0603Metric, F.Cu at (97.8, 49.0)
- added C18: 0.1uF, Capacitor_SMD:C_0201_0603Metric, F.Cu at (97.8, 50.7)
- added J1: Micro_SD_Card_Det_Hirose_DM3AT, Connector_Card:microSD_HC_Hirose_DM3AT-SF-PEJM5, F.Cu at (104.9, 55.7)
- added J3: Conn_01x02_Pin, Connector_PinHeader_1.00mm:PinHeader_1x02_P1.00mm_Vertical, F.Cu at (100.7, 47.9)
- added R12: 10kR, Resistor_SMD:R_0201_0603Metric, F.Cu at (114.5, 50.7)
- added R13: 10kR, Resistor_SMD:R_0201_0603Metric, F.Cu at (114.5, 52.5)
- added R14: 10kR, Resistor_SMD:R_0201_0603Metric, F.Cu at (114.5, 54.2)
- added R15: 10kR, Resistor_SMD:R_0201_0603Metric, F.Cu at (114.5, 56.0)
- added R16: 10kR, Resistor_SMD:R_0201_0603Metric, F.Cu at (114.5, 57.7)
- added R17: 100KR, Resistor_SMD:R_0201_0603Metric, F.Cu at (97.8, 52.5)
- added R18: 1MR, Resistor_SMD:R_0201_0603Metric, F.Cu at (97.8, 54.2)
- added R19: 100KR, Resistor_SMD:R_0201_0603Metric, F.Cu at (97.8, 56.0)
- added R20: 100KR, Resistor_SMD:R_0201_0603Metric, F.Cu at (97.8, 57.7)
- added R21: 100KR, Resistor_SMD:R_0201_0603Metric, F.Cu at (97.8, 59.5)
- added U9: LMV358IDR, footprints:LMV358IDR, F.Cu at (100.8, 49.7)
Connections:
- U1 pad 19: /IO15 -> /J1_CD
- U1 pad 20: /IO16 -> /J1_CMD
- U1 pad 21: /IO17 -> /J1_DAT0
- U1 pad 22: /IO18 -> /J1_DET_A
- U1 pad 25: /IO21 -> unconnected-(U1-IO21-Pad25)

Commit message: new library
Parts:
- removed J1: Micro_SD_Card_Det_Hirose_DM3AT, Connector_Card:microSD_HC_Hirose_DM3AT-SF-PEJM5
- added J4: 5033981892, footprints:CONN_503398-1892_MOL, F.Cu at (104.7, 71.5)

Commit message: change so much
Parts:
- added J1: Conn_01x01_Pin, Connector_PinHeader_1.00mm:PinHeader_1x01_P1.00mm_Vertical, F.Cu at (70.1, 60.9)
- added J5: Conn_01x02_Pin, Connector_PinHeader_1.00mm:PinHeader_1x02_P1.00mm_Vertical, B.Cu at (75.1, 40.4)
- added J6: Conn_01x01_Pin, Connector_PinHeader_1.00mm:PinHeader_1x01_P1.00mm_Vertical, F.Cu at (70.1, 63.9)
- C14, C15, C16, C17, C18, C3, R12, R13, R14, R15, R16, R17, R18, R19, R20, R21, U9: moved to B.Cu
- moved J4 48.1 mm to (75.4, 33.3), turned to 180 degrees
- moved R16 37.9 mm to (84.5, 34.7), turned to -90 degrees
- moved R15 37.8 mm to (84.5, 33.0), turned to -90 degrees
- moved R14 37.8 mm to (84.5, 31.3), turned to -90 degrees
- moved R13 37.8 mm to (84.5, 29.6), turned to -90 degrees
- moved R12 34.8 mm to (83.6, 34.7), turned to -90 degrees
- moved C15 34.8 mm to (83.6, 33.0), turned to -90 degrees
- moved C14 34.8 mm to (83.6, 31.3), turned to -90 degrees
- moved R21 31.0 mm to (81.7, 33.0), turned to -90 degrees
- moved R20 31.0 mm to (81.7, 31.3), turned to -90 degrees
- moved R18 29.0 mm to (82.7, 29.5), turned to -90 degrees
- moved R19 26.7 mm to (81.7, 34.7), turned to -90 degrees
- moved R17 26.0 mm to (82.7, 31.3), turned to -90 degrees
- moved C3 23.9 mm to (81.7, 29.5), turned to -90 degrees
- moved C18 23.3 mm to (82.7, 33.0), turned to -90 degrees
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Connections:
- U1 pad 10: /IO6 -> /OUT_A
- U1 pad 11: /IO7 -> /OUT_B
- U1 pad 25: unconnected-(U1-IO21-Pad25) -> /Temp_SDA
- U1 pad 26: /IO26 -> /Temp_SCL
Routing:
- net Net-(U4-ILIM): track 0.00 -> 233.5 mm, vias 0 -> 2
- net GND: track 0.00 -> 214.0 mm, vias 0 -> 3
- net +3V3: track 0.00 -> 131.7 mm, vias 0 -> 11
- net /J1_CMD: track 0.00 -> 53.4 mm, vias 0 -> 2
- net /VBUS: track 0.00 -> 50.5 mm, vias 0 -> 4
- net /OUT_B: track 0.00 -> 49.1 mm, vias 0 -> 3
- net /J1_DAT0: track 0.00 -> 42.5 mm, vias 0 -> 3
- net /J1_CD: track 0.00 -> 40.9 mm, vias 0 -> 2
- net /skin++: track 0.00 -> 38.3 mm, vias 0 -> 2
- net /OUT_A: track 0.00 -> 37.2 mm, vias 0 -> 3
- net /~{PGOOD}: track 0.00 -> 28.0 mm, vias 0 -> 2
- net /U1_BAT: track 0.00 -> 25.8 mm, vias 0 -> 3
- net /USB_D+: track 0.00 -> 24.6 mm, vias 0 -> 3
- net /VREF: track 0.00 -> 23.2 mm, vias 0 -> 2
- net /D+: track 0.00 -> 21.7 mm, vias 0 -> 2
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Other:
- board size 16.8 x 23.9 mm -> 18.2 x 40.8 mm
- copper layers 2 -> 4

Commit message: placement and routing
Routing:
- net Net-(U4-ILIM): track 233.5 -> 24.5 mm
- net GND: track 214.0 -> 58.7 mm, vias 3 -> 11
- net +3V3: track 131.7 -> 32.7 mm, vias 11 -> 16
- net /OUT_B: track 49.1 -> 93.1 mm, vias 3 -> 7
- net /J1_DAT0: track 42.5 -> 65.7 mm, vias 3 -> 5
- net /USB_D-: track 0.00 -> 20.7 mm, vias 0 -> 3
- net /U3_SDX: track 14.9 -> 33.5 mm, vias 2 -> 5
- net /~{CE}: track 21.6 -> 36.4 mm, vias 2 -> 1
- net /VREF: track 23.2 -> 9.61 mm
- net /Temp_SDA: track 17.9 -> 30.0 mm, vias 1 -> 0
- net /U3_SCX: track 14.0 -> 24.7 mm, vias 2 -> 4
- net /~{PGOOD}: track 28.0 -> 17.4 mm
- net /J1_CD: track 40.9 -> 32.1 mm, vias 2 -> 3
- net /OUT_A: track 37.2 -> 45.5 mm, vias 3 -> 6
- net /VBUS: track 50.5 -> 42.6 mm, vias 4 -> 7
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- added copper zone on In2.Cu, net +3V3
- added copper zone on B.Cu, net GND
- added copper zone on In1.Cu, net GND

Commit message: placement and routing
Parts:
- moved J5 25.1 mm to (84.2, 63.8), turned to 180 degrees
Routing:
- net /OUT_B: track 93.1 -> 40.9 mm, vias 7 -> 5
- net /D-: track 28.2 -> 62.6 mm, vias 2 -> 5
- net GND: track 58.7 -> 90.5 mm, vias 11 -> 25
- net /Temp_SDA: track 30.0 -> 9.95 mm
- net /U3_SDX: track 33.5 -> 15.4 mm, vias 5 -> 1
- net /J1_DAT0: track 65.7 -> 48.9 mm, vias 5 -> 3
- net /U1_BAT: track 27.1 -> 43.3 mm, vias 4 -> 6
- net /OUT_A: track 45.5 -> 61.0 mm, vias 6 -> 3
- net /D+: track 25.1 -> 39.7 mm, vias 7 -> 5
- net /Temp_SCL: track 26.3 -> 11.9 mm
- net /VLDO: track 14.3 -> 27.6 mm
- net /~{CE}: track 36.4 -> 24.3 mm, vias 1 -> 5
- net /U3_SCX: track 24.7 -> 13.1 mm, vias 4 -> 1
- net /~{CHG}: track 20.8 -> 11.6 mm
- net /~{PGOOD}: track 17.4 -> 8.91 mm
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- removed copper zone on B.Cu, net GND

Commit message: route maxing
Routing:
- net GND: track 90.5 -> 0.00 mm, vias 25 -> 0
- net /D-: track 62.6 -> 0.00 mm, vias 5 -> 0
- net /OUT_A: track 61.0 -> 0.00 mm, vias 3 -> 0
- net /J1_CMD: track 60.7 -> 0.00 mm, vias 4 -> 0
- net /J1_DAT0: track 48.9 -> 0.00 mm, vias 3 -> 0
- net /U1_BAT: track 43.3 -> 0.00 mm, vias 6 -> 0
- net /VBUS: track 43.0 -> 0.00 mm, vias 9 -> 0
- net /OUT_B: track 40.9 -> 0.00 mm, vias 5 -> 0
- net /J1_CD: track 39.9 -> 0.00 mm, vias 5 -> 0
- net /D+: track 39.7 -> 0.00 mm, vias 5 -> 0
- net /skin++: track 36.7 -> 0.00 mm
- net Net-(U4-ILIM): track 29.1 -> 0.00 mm, vias 2 -> 0
- net /VLDO: track 27.6 -> 0.00 mm, vias 4 -> 0
- net Net-(U4-ISET): track 24.9 -> 0.00 mm, vias 2 -> 0
- net +3V3: track 24.9 -> 0.00 mm, vias 17 -> 0
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- removed copper zone on In2.Cu, net +3V3
- removed copper zone on In1.Cu, net GND
